Commit message: added proper blimp dimentions

File: assets/blimp/urdf/blimp.urdf (robot description, URDF)
Before this commit: robot blimp, 15 links, 14 joints
Links:
- link base: mass 1.66 -> 4.622; geometry collision cylinder length=3.5 radius=0.9; visual mesh filename=../meshes/blimp_body/blimp_body_v4.dae scale=1 1 1
- link blimp_rud_bot: mass 0.02 -> 0.3
- link blimp_rud_left: mass 0.02 -> 0.3
- link blimp_rud_right: mass 0.02 -> 0.3
- link blimp_rud_top: mass 0.02 -> 0.3
- link blimp_stick: mass 0.01 -> 0.2
- link blimp_support1: mass 0.0 -> None; geometry visual mesh filename=../meshes/blimp_support/blimp_support_v5.dae scale=1.0 1.0 1.0
- link blimp_support2: mass 0.0 -> None; geometry visual mesh filename=../meshes/blimp_support/blimp_support_v5.dae scale=1.0 1.0 1.0
- link gondola: mass 0.5 -> 2.605; geometry collision box size=0.32 0.16 0.2; visual mesh filename=../meshes/blimp_gondola/blimp_gondola_v4.dae scale=1 1 1
- link rud_bot: mass 0.02 -> 0.07
- link rud_left: mass 0.02 -> 0.07
- link rud_right: mass 0.02 -> 0.07
- link rud_top: mass 0.02 -> 0.07
Joints:
- joint base_rud_bot: origin xyz=-1.4 0 -0.75 rpy=0 0.164533 0 -> xyz=-1.55 0 -0.85 rpy=0 0.164533 0
- joint base_rud_left: origin xyz=-1.4 0.75 0.05 rpy=1.57075 0 0.174533 -> xyz=-1.55 0.85 0.05 rpy=1.57075 0 0.174533
- joint base_rud_right: origin xyz=-1.4 -0.75 0.05 rpy=-1.57075 0 -0.174533 -> xyz=-1.55 -0.85 0.05 rpy=-1.57075 0 -0.174533
- joint base_rud_top: origin xyz=-1.4 0 0.75 rpy=3.14159 -0.164533 0 -> xyz=-1.55 0 0.85 rpy=3.14159 -0.164533 0
- joint gondola_stick: origin xyz=0.9 0 -1.06 rpy=1.57075 0 0 -> xyz=1.06 0 -1.12 rpy=1.57075 0 0
