Commit message: pm2d rand

File: assets/urdf/pointer.urdf (robot description, URDF)
Before this commit: robot thepointer, 2 links, 1 joints
Links:
- removed link pointer
- added link pointer_body, mass 0.5; collision mesh filename=../mesh/pointer.dae scale=0.4 0.4 0.4; visual mesh filename=../mesh/pointer.dae scale=0.4 0.4 0.4
- link base_link: geometry collision mesh filename=../mesh/pointer.dae scale=0.4 0.4 0.4; visual mesh filename=../mesh/pointer.dae scale=0.4 0.4 0.4
Joints:
- joint base_to_pointer: child pointer -> pointer_body
